Commit message: Added

File: mujoco/models/motor_test/test.urdf (robot description, URDF)
Before this commit: robot Test, 4 links, 3 joints
Links:
- added link load_1, mass 0.3143757525105692; collision mesh filename=/meshes/load_1.stl scale=0.001 0.001 0.001; visual mesh filename=/meshes/load_1.stl scale=0.001 0.001 0.001
Joints:
- added joint Rigid 4: type fixed, parent shaft_1, child load_1, origin xyz=2e-06 8e-05 0.6 rpy=0 0 0
